File: keyboard/keyboard.sch (KiCad schematic (older format))
At the start: 29 parts, among them J1 USB_C_Receptacle_USB2.0, J2 USB_C_Receptacle_USB2.0, K1 KEYSW, K2 KEYSW, K3 KEYSW, K4 KEYSW, SW1 SW_PUSH, U1 ATMEGA32U4, U2 USB2514B_Bi, U3 FT232RL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

Commit message: [0.0.3]
Parts:
- removed D1, D2, D3, D4: D, symbol Device:D
- removed J1: USB_C_Receptacle_USB2.0, symbol Connector:USB_C_Receptacle_USB2.0
- removed K1, K2, K3, K4: KEYSW, symbol keyboard_parts:KEYSW
- added R? (x2): 100k, symbol Device:R
- added R? (x2): 10k, symbol Device:R
Connections:
- net +5V: now also J2.A1 (GND), J2.A12 (GND), J2.B1 (GND), J2.B12 (GND), J2.S1 (SHIELD), U2.37 (VSS)
- net col0: now also U1.36 (PF7); no longer U1.39 (PF4)
- net col1: now also U1.32 (PC7); no longer U1.38 (PF5)
- net col5: now reaches U1.10 (PB2/MOSI)
- net col6: now reaches U1.11 (PB3/MISO)
- net col10: now reaches U1.12 (PB7/~RTS)
- net reset: now reaches R1.1, SW1.2, U1.13 (~RESET)
- net reset: now also U2.26 (RESET_N)
- net col11: now reaches U1.18 (PD0/INT0)
- net col12: now reaches U1.19 (PD1/INT1)
- net at U1.2 (UVcc): now also U2.23 (VDD33)
- net col13: now reaches U1.20 (PD2/RXD1)
- net col7: now reaches U1.28 (PB4)
- net col8: now reaches U1.29 (PB5)
- net col9: now reaches U1.30 (PB6)
- net col2: now reaches U1.31 (PC6)
- net row4: now reaches U1.37 (PF6)
- net col3: now reaches U1.8 (PB0/SS)
- net col4: now reaches U1.9 (PB1/SCK)
- net at U2.15 (VDD33): now also R?.1, R?.1
- net at U2.24 (SCL/SMBCLK/CFG_SEL0): now also R?.2
- net at U2.25 (HS_IND/CFG_SEL1): now also R?.2
- net at U2.27 (VBUS_DET): now also R?.1, R?.1
- net at U2.30 (USBDM_UP): now also J2.A7 (D-)
- net at U2.31 (USBDP_UP): now also J2.A6 (D+)
- net at R3.1: now also J2.A4 (VBUS), J2.A9 (VBUS), J2.B4 (VBUS), J2.B9 (VBUS), R?.2, R?.2
- new net row2: U1.39 (PF4)
- new net row3: U1.38 (PF5)
- no-connect marks 36 -> 28
Other:
- note added: "Connect clock here"
- note added: "Tie high"
- note added: "Tie low\n"
- moved on the sheet: C1, C2, C3, C4, C5, C6, C7, C8, J2, R1, R2, R3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
